File: hardware/pb1000_emulator.kicad_sch (KiCad schematic)
At the start: 2 parts, among them U1 Raspberry Pi Pico 2

Commit message: 機能実装おおむねFIX。テスト・調整フェーズ
Parts:
- removed LCD1: ILI9341 320x240, symbol Connector:LCD_ILI9341
- U1: value Raspberry Pi Pico 2 -> Raspberry Pi Pico 2 (RP2350)
Other:
- note added: "=== Beep Output (PWM) ==="
- note added: "=== Console UART (UART1) ==="
- note added: "=== GPIO Summary ==="
- note added: "=== ILI9341 320x240 TFT LCD ==="
- note added: "=== Joystick Input (direct, PULL_UP, active LOW) ==="
- note added: "=== PIO UART -- Virtual RS-232C ==="
- note added: "=== SD Card Module (SPI1) ==="
- note added: "=== SPI1 Shared Bus ==="
- note added: "=== Touch Panel XPT2046 (SPI1) ==="
- note added: "=== USB Keyboard ==="
- note added: "All GPIO pins are 3.3V logic. Do NOT apply 5V signals directly to Pico 2 pins."
- note added: "Baudrate: default 115200. Configurable via pb1000.ini [keyboard] uart_baudrate."
- note added: "Baudrate: default 9600. Configurable via pb1000.ini [pio_uart] baudrate."
- note added: "Default: freq=4470 Hz, duty=30%. Configurable via pb1000.ini [beep]."
- note added: "GP10 = SCK (SPI1 Clock -- shared: LCD / SD / Touch)"
- note added: "GP10 SPI1_SCK (shared) GP11 SPI1_MOSI (shared)"
- note added: "GP10/GP11/GP12: SCK/MOSI/MISO (SPI1 shared)"
- note added: "GP10/GP11/GP12: T_CLK/T_DIN/T_DO (SPI1 shared)"
- note added: "GP11 = MOSI (SPI1 TX -- shared: LCD / SD / Touch)"
- note added: "GP12 = MISO (SPI1 RX -- shared: LCD / SD / Touch)"
- note added: "GP12 SPI1_MISO (shared) GP13 PIO_RX RS-232C"
- note added: "GP13 = PIO_RX (RS-232C RX -- to external TX)"
- note added: "GP14 = BEEP_PWM (PWM -- connect via 100 ohm to piezo buzzer or small speaker)"
- note added: "GP14 BEEP_PWM Buzzer GP15 SD_CS SD Card"
- note added: "GP15 = SD_CS (Chip Select)"
- note added: "GP16 = T_CS (Chip Select)"
- note added: "GP16 T_CS XPT2046 GP17 T_IRQ XPT2046"
- note added: "GP17 = T_IRQ (Touch Interrupt -- active LOW, input with pull-up)"
- note added: "GP18 = JOY_UP -- default: KEY_UP"
- note added: "GP18 JOY_UP Joystick GP19 JOY_DOWN Joystick"
- note added: "GP19 = JOY_DOWN -- default: KEY_DOWN"
- note added: "GP20 = JOY_LEFT -- default: KEY_LEFT"
- note added: "GP20 JOY_LEFT Joystick GP21 JOY_RIGHT Joystick"
- note added: "GP21 = JOY_RIGHT -- default: KEY_RIGHT"
- note added: "GP22 = LCD_BL (Backlight -- connect via 100 ohm to 3.3V or VBUS)"
- note added: "GP22 LCD_BL ILI9341 BL GP26 JOY_FIRE1 Joystick"
- note added: "GP26 = JOY_FIRE1 -- default: EXE"
- note added: "GP27 = JOY_FIRE2 -- default: SHIFT"
- note added: "GP27 JOY_FIRE2 Joystick"
- note added: "GP4 = UART1_TX (to PC RX -- debug / REPL / keyboard input)"
- note added: "GP4 UART1_TX Console GP5 UART1_RX Console"
- note added: "GP5 = UART1_RX (to PC TX)"
- note added: "GP6 = PIO_TX (RS-232C TX -- to external RX)"
- note added: "GP6 PIO_TX RS-232C GP7 LCD_RST ILI9341"
- note added: "GP7 = LCD_RST (Reset -- active LOW)"
- note added: "GP8 = LCD_DC (Data / Command)"
- note added: "GP8 LCD_DC ILI9341 GP9 LCD_CS ILI9341"
- note added: "GP9 = LCD_CS (Chip Select)"
- note added: "Key mapping configurable via pb1000.ini [joystick]. See references/joystick_3bit_encoding_circuit.md for encoder option."
- note added: "Micro-USB port via OTG adapter -- connect standard USB HID keyboard."
- note added: "NOTE: 3.3V logic. Use MAX3232 or similar for true RS-232C voltage levels."
- note removed: "See doc/hardware_guide.md for full pin table."
- moved on the sheet: U1
Changed lines of the file:
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@@
 (kicad_sch (version 20230121) (generator kicad_sch_editor)
-  (paper "A4")
+  (paper "A3")
   (title_block
     (title "PB-1000 Emulator (Raspberry Pi Pico 2)")
     (company "Antigravity AI")
-    (comment 1 "Wiring Guide for ILI9341, SD Card, Touch, and USB")
+    (date "2026-05-30")
+    (comment 1 "Wiring Guide: ILI9341 / SD Card / XPT2046 / UART / PIO UART / Beep / Joystick")
+    (comment 2 "All SPI devices share SPI1 (GP10 SCK / GP11 MOSI / GP12 MISO). CS pins are independent.")
+    (comment 3 "See doc/hardware_guide.md for full details.")
   )
-  (symbol (lib_id "Pico2:Raspberry_Pi_Pico_2") (at 100 100 0) (unit 1)
+  (symbol (lib_id "Pico2:Raspberry_Pi_Pico_2") (at 60 120 0) (unit 1)
     (in_bom yes) (on_board yes) (fields_autoplaced)
-    (property "Reference" "U1" (id 0) (at 100 73.66 0))
-    (property "Value" "Raspberry Pi Pico 2" (id 1) (at 100 71.12 0))
+    (property "Reference" "U1" (id 0) (at 60 93 0))
+    (property "Value" "Raspberry Pi Pico 2 (RP2350)" (id 1) (at 60 90.5 0))
   )
-  (symbol (lib_id "Connector:LCD_ILI9341") (at 180 80 0) (unit 1)
-    (in_bom yes) (on_board yes) (fields_autoplaced)
-    (property "Reference" "LCD1" (id 0) (at 180 67.31 0))
-    (property "Value" "ILI9341 320x240" (id 1) (at 180 64.77 0))
+  (text "=== SPI1 Shared Bus ===" (at 130 60 0)
+    (effects (font (size 2.5 2.5) (bold yes)) (justify left))
   )
-  (label "GP10 (SCK1)" (at 110.16 100.33 0)
-    (effects (font (size 1.27 1.27)) (justify left))
+  (text "GP10 = SCK    (SPI1 Clock  -- shared: LCD / SD / Touch)" (at 130 65 0)
+    (effects (font (size 1.5 1.5)) (justify left))
   )
-  (label "GP11 (TX1)" (at 110.16 102.87 0)
-    (effects (font (size 1.27 1.27)) (justify left))
+  (text "GP11 = MOSI   (SPI1 TX    -- shared: LCD / SD / Touch)" (at 130 68.5 0)
+    (effects (font (size 1.5 1.5)) (justify left))
   )
-  (label "GP12 (RX1)" (at 110.16 105.41 0)
-    (effects (font (size 1.27 1.27)) (justify left))
+  (text "GP12 = MISO   (SPI1 RX    -- shared: LCD / SD / Touch)" (at 130 72 0)
+    (effects (font (size 1.5 1.5)) (justify left))
   )
-  (label "GP9 (LCD_CS)" (at 110.16 107.95 0)
-    (effects (font (size 1.27 1.27)) (justify left))
+  (text "=== ILI9341 320x240 TFT LCD ===" (at 130 82 0)
+    (effects (font (size 2.5 2.5) (bold yes)) (justify left))
   )
-  (label "GP8 (LCD_DC)" (at 110.16 110.49 0)
-    (effects (font (size 1.27 1.27)) (justify left))
+  (text "GP9  = LCD_CS    (Chip Select)" (at 130 87 0)
+    (effects (font (size 1.5 1.5)) (justify left))
   )
-  (label "GP7 (LCD_RST)" (at 110.16 113.03 0)
-    (effects (font (size 1.27 1.27)) (justify left))
+  (text "GP8  = LCD_DC    (Data / Command)" (at 130 90.5 0)
+    (effects (font (size 1.5 1.5)) (justify left))
   )
-  (label "GP15 (SD_CS)" (at 110.16 115.57 0)
-    (effects (font (size 1.27 1.27)) (justify left))
+  (text "GP7  = LCD_RST   (Reset -- active LOW)" (at 130 94 0)
+    (effects (font (size 1.5 1.5)) (justify left))
   )
-  (label "GP16 (T_CS)" (at 110.16 118.11 0)
-    (effects (font (size 1.27 1.27)) (justify left))
+  (text "GP22 = LCD_BL    (Backlight -- connect via 100 ohm to 3.3V or VBUS)" (at 130 97.5 0)
+    (effects (font (size 1.5 1.5)) (justify left))
   )
-  (text "See doc/hardware_guide.md for full pin table." (at 100 150 0)
-    (effects (font (size 3 3)) (justify left))
+  (text "GP10/GP11/GP12: SCK/MOSI/MISO (SPI1 shared)" (at 130 101 0)
+    (effects (font (size 1.5 1.5)) (justify left))
+  )
+  (text "=== SD Card Module (SPI1) ===" (at 130 111 0)
+    (effects (font (size 2.5 2.5) (bold yes)) (justify left))
+  )
+  (text "GP15 = SD_CS     (Chip Select)" (at 130 116 0)
+    (effects (font (size 1.5 1.5)) (justify left))
+  )
+  (text "GP10/GP11/GP12: SCK/MOSI/MISO (SPI1 shared)" (at 130 119.5 0)
+    (effects (font (size 1.5 1.5)) (justify left))
+  )
+  (text "=== Touch Panel XPT2046 (SPI1) ===" (at 130 129.5 0)
+    (effects (font (size 2.5 2.5) (bold yes)) (justify left))
+  )
+  (text "GP16 = T_CS      (Chip Select)" (at 130 134.5 0)
+    (effects (font (size 1.5 1.5)) (justify left))
+  )
+  (text "GP17 = T_IRQ     (Touch Interrupt -- active LOW, input with pull-up)" (at 130 138 0)
+    (effects (font (size 1.5 1.5)) (justify left))
+  )
+  (text "GP10/GP11/GP12: T_CLK/T_DIN/T_DO (SPI1 shared)" (at 130 141.5 0)
+    (effects (font (size 1.5 1.5)) (justify left))
+  )
+  (text "=== Console UART (UART1) ===" (at 130 151.5 0)
+    (effects (font (size 2.5 2.5) (bold yes)) (justify left))
+  )
+  (text "GP4  = UART1_TX  (to PC RX -- debug / REPL / keyboard input)" (at 130 156.5 0)
+    (effects (font (size 1.5 1.5)) (justify left))
+  )
+  (text "GP5  = UART1_RX  (to PC TX)" (at 130 160 0)
+    (effects (font (size 1.5 1.5)) (justify left))
+  )
+  (text "Baudrate: default 115200. Configurable via pb1000.ini [keyboard] uart_baudrate." (at 130 163.5 0)
+    (effects (font (size 1.5 1.5)) (justify left))
+  )
+  (text "=== PIO UART -- Virtual RS-232C ===" (at 130 173.5 0)
+    (effects (font (size 2.5 2.5) (bold yes)) (justify left))
+  )
+  (text "GP6  = PIO_TX    (RS-232C TX -- to external RX)" (at 130 178.5 0)
+    (effects (font (size 1.5 1.5)) (justify left))
+  )
+  (text "GP13 = PIO_RX    (RS-232C RX -- to external TX)" (at 130 182 0)
+    (effects (font (size 1.5 1.5)) (justify left))
+  )
+  (text "Baudrate: default 9600. Configurable via pb1000.ini [pio_uart] baudrate." (at 130 185.5 0)
+    (effects (font (size 1.5 1.5)) (justify left))
+  )
+  (text "NOTE: 3.3V logic. Use MAX3232 or similar for true RS-232C voltage levels." (at 130 189 0)
+    (effects (font (size 1.5 1.5)) (justify left))
+  )
+  (text "=== Beep Output (PWM) ===" (at 130 199 0)
+    (effects (font (size 2.5 2.5) (bold yes)) (justify left))
+  )
+  (text "GP14 = BEEP_PWM  (PWM -- connect via 100 ohm to piezo buzzer or small speaker)" (at 130 204 0)
+    (effects (font (size 1.5 1.5)) (justify left))
+  )
+  (text "Default: freq=4470 Hz, duty=30%. Configurable via pb1000.ini [beep]." (at 130 207.5 0)
+    (effects (font (size 1.5 1.5)) (justify left))
+  )
+  (text "=== Joystick Input (direct, PULL_UP, active LOW) ===" (at 130 217.5 0)
+    (effects (font (size 2.5 2.5) (bold yes)) (justify left))
+  )
+  (text "GP18 = JOY_UP    -- default: KEY_UP" (at 130 222.5 0)
+    (effects (font (size 1.5 1.5)) (justify left))
+  )
+  (text "GP19 = JOY_DOWN  -- default: KEY_DOWN" (at 130 226 0)
+    (effects (font (size 1.5 1.5)) (justify left))
+  )
+  (text "GP20 = JOY_LEFT  -- default: KEY_LEFT" (at 130 229.5 0)
+    (effects (font (size 1.5 1.5)) (justify left))
+  )
+  (text "GP21 = JOY_RIGHT -- default: KEY_RIGHT" (at 130 233 0)
+    (effects (font (size 1.5 1.5)) (justify left))
+  )
+  (text "GP26 = JOY_FIRE1 -- default: EXE" (at 130 236.5 0)
+    (effects (font (size 1.5 1.5)) (justify left))
+  )
+  (text "GP27 = JOY_FIRE2 -- default: SHIFT" (at 130 240 0)
+    (effects (font (size 1.5 1.5)) (justify left))
+  )
+  (text "Key mapping configurable via pb1000.ini [joystick]. See references/joystick_3bit_encoding_circuit.md for encoder option." (at 130 243.5 0)
+    (effects (font (size 1.5 1.5)) (justify left))
+  )
+  (text "=== USB Keyboard ===" (at 130 253.5 0)
+    (effects (font (size 2.5 2.5) (bold yes)) (justify left))
+  )
+  (text "Micro-USB port via OTG adapter -- connect standard USB HID keyboard." (at 130 258.5 0)
+    (effects (font (size 1.5 1.5)) (justify left))
+  )
+  (text "=== GPIO Summary ===" (at 130 268.5 0)
+    (effects (font (size 2.5 2.5) (bold yes)) (justify left))
+  )
+  (text "GP4  UART1_TX Console    GP5  UART1_RX Console" (at 130 273.5 0)
+    (effects (font (size 1.5 1.5)) (justify left))
+  )
+  (text "GP6  PIO_TX  RS-232C     GP7  LCD_RST ILI9341" (at 130 277 0)
+    (effects (font (size 1.5 1.5)) (justify left))
+  )
+  (text "GP8  LCD_DC  ILI9341     GP9  LCD_CS  ILI9341" (at 130 280.5 0)
+    (effects (font (size 1.5 1.5)) (justify left))
+  )
+  (text "GP10 SPI1_SCK (shared)   GP11 SPI1_MOSI (shared)" (at 130 284 0)
+    (effects (font (size 1.5 1.5)) (justify left))
+  )
+  (text "GP12 SPI1_MISO (shared)  GP13 PIO_RX  RS-232C" (at 130 287.5 0)
+    (effects (font (size 1.5 1.5)) (justify left))
+  )
+  (text "GP14 BEEP_PWM Buzzer     GP15 SD_CS   SD Card" (at 130 291 0)
+    (effects (font (size 1.5 1.5)) (justify left))
+  )
+  (text "GP16 T_CS    XPT2046     GP17 T_IRQ   XPT2046" (at 130 294.5 0)
+    (effects (font (size 1.5 1.5)) (justify left))
+  )
+  (text "GP18 JOY_UP  Joystick    GP19 JOY_DOWN Joystick" (at 130 298 0)
+    (effects (font (size 1.5 1.5)) (justify left))
+  )
+  (text "GP20 JOY_LEFT Joystick   GP21 JOY_RIGHT Joystick" (at 130 301.5 0)
+    (effects (font (size 1.5 1.5)) (justify left))
+  )
+  (text "GP22 LCD_BL  ILI9341 BL  GP26 JOY_FIRE1 Joystick" (at 130 305 0)
+    (effects (font (size 1.5 1.5)) (justify left))
+  )
+  (text "GP27 JOY_FIRE2 Joystick" (at 130 308.5 0)
+    (effects (font (size 1.5 1.5)) (justify left))
+  )
+  (text "All GPIO pins are 3.3V logic. Do NOT apply 5V signals directly to Pico 2 pins." (at 130 318.5 0)
+    (effects (font (size 1.5 1.5)) (justify left))
   )
 )
